File: CM5_MINIMA_3.kicad_pcb (KiCad board)
At the start: 6 copper layers, 54.6 x 57.1 mm, 101 parts, among them J101 TYPEC-305-ACP16H458, J501 GT-HD001B-CNNG1, J502 I2C, J503 SPI, J601 JST_SHBM04B-SRSS-TB, J701 Bus_M.2_Socket_M, J802 Conn_01x22_Female, M701 M.2 Solder Nut, M702 M.2 Solder Nut, SW101 MK-11C04-G013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

Commit message: arcs
Parts:
- added H102: MountingHole_Pad, MountingHole:MountingHole_2.7mm_Pad, F.Cu at (78.2, 23.4)
- added H103: MountingHole_Pad, MountingHole:MountingHole_2.7mm_Pad, F.Cu at (133.2, 23.4)
- added H104: MountingHole_Pad, MountingHole:MountingHole_2.7mm_Pad, F.Cu at (133.2, 81.3)
- added H105: MountingHole_Pad, MountingHole:MountingHole_2.7mm_Pad, F.Cu at (78.2, 81.3)
- moved TP104 4.05 mm to (126.9, 25.1)
Other:
- board size 54.6 x 57.1 mm -> 61.2 x 64.2 mm

Commit message: vias
Parts:
- removed kibuzzard-6775AD68: G***, kibuzzard-6775AD68
- removed kibuzzard-67D06071: G***, kibuzzard-67D06071
- added C503: 100n, Capacitor_SMD:C_0402_1005Metric, B.Cu at (84.6, 74.5)
- added R107: 10k, Resistor_SMD:R_0402_1005Metric, B.Cu at (81.6, 73.7)
- added R108: 10k, Resistor_SMD:R_0402_1005Metric, B.Cu at (82.9, 78.2)
- added U1: LIS3DH, Package_LGA:LGA-16_3x3mm_P0.5mm_LayoutBorder3x5y, B.Cu at (82.4, 76.0)
- added kibuzzard-67EBB9C1: G***, kibuzzard-67EBB9C1, F.Cu at (95.8, 55.2)
- added kibuzzard-67EBD21C: G***, kibuzzard-67EBD21C, B.Cu at (86.6, 76.0)
- added kibuzzard-67EBD221: G***, kibuzzard-67EBD221, B.Cu at (82.4, 79.7)
- added kibuzzard-67EBD321: G***, kibuzzard-67EBD321, F.Cu at (122.0, 61.9)
- C702: footprint Capacitor_Tantalum_SMD:CP_EIA-7343-31_Kemet-D -> Capacitor_Tantalum_SMD:CP_EIA-3528-21_Kemet-B; moved to F.Cu
- moved TP104 8.33 mm to (129.6, 33.0)
- moved C702 5.31 mm to (82.5, 68.8)
- moved TP106 3.65 mm to (109.5, 60.2)
- moved kibuzzard-6773B9F7 2.37 mm to (128.2, 62.0)
Connections:
- net Net-(U702-LX) renamed /PCIe-M2/M2_LX
Routing:
- net Net-(U1-CS): track 0.00 -> 6.86 mm
- net +3V3_PI: track 131.3 -> 138.1 mm
- net VBUS_USB2.0: track 22.9 -> 18.4 mm, vias 2 -> 0
- net /SDA: track 68.3 -> 71.6 mm, vias 3 -> 4
- net /SCL: track 65.2 -> 67.7 mm, vias 3 -> 4
- net M2_3V3: track 95.3 -> 97.4 mm
- net Net-(U1-SDO): track 0.00 -> 1.01 mm
- net GND: vias 171 -> 257
- added copper zone on F.Cu, net /PCIe-M2/M2_LX
Other:
- outline, holes or cut-outs redrawn
- board text removed: "R3.1"

Commit message: DRC and prod files
Parts:
- removed R105, R106: 0R, Resistor_SMD:R_0402_1005Metric
- removed kibuzzard-67758943: G***, kibuzzard-67758943
- removed kibuzzard-67EBD321: G***, kibuzzard-67EBD321
- added CN1: SM02B-SRSS-TB (LF)(SN), EasyEDA:CONN-SMD_2P-P1.00_SM02B-SRSS-TB-LF-SN, B.Cu at (83.2, 69.5)
- added kibuzzard-67EBEF55: G***, kibuzzard-67EBEF55, F.Cu at (121.5, 62.4)
- added kibuzzard-67EBF015: G***, kibuzzard-67EBF015, B.Cu at (80.0, 62.4)
- added kibuzzard-67EBF0A0: G***, kibuzzard-67EBF0A0, B.Cu at (88.1, 69.0)
- added kibuzzard-67EBF14E: G***, kibuzzard-67EBF14E, B.Cu at (81.7, 72.1)
- moved C709 3.92 mm to (119.0, 67.8), turned to 180 degrees
- moved TP106 3.54 mm to (106.2, 61.5)
Connections:
- J701 pad 20: /PCIe-M2/TX -> unconnected-(J701-NC-Pad20)
- J701 pad 22: /PCIe-M2/RX -> unconnected-(J701-NC-Pad22)
- Module301 pad 76: /CM5/VBAT -> +BATT
Routing:
- net +BATT: track 0.00 -> 69.0 mm, vias 0 -> 4
- net /CM5/GPIO4: track 30.9 -> 0.00 mm, vias 1 -> 0
- net /CM5/GPIO5: track 27.6 -> 0.00 mm, vias 1 -> 0
- net +3V3_PI: track 138.1 -> 142.2 mm, vias 10 -> 12
- net /PCIe-M2/TX: track 3.69 -> 0.00 mm
- net /PCIe-M2/RX: track 3.68 -> 0.00 mm
- net /CM5/PCIE_PI.PWR_EN: track 48.1 -> 49.7 mm
- net /SDA: track 71.6 -> 70.9 mm
- net /CM5/CAM_GPIO0: track 27.4 -> 26.8 mm
- net GND: vias 257 -> 256
