File: CM5_MINIMA_3.kicad_pcb (KiCad board)
At the start: 6 copper layers, 61.2 x 64.2 mm, 112 parts, among them CN1 SM02B-SRSS-TB (LF)(SN), J1 GLPLX-SMT-188S7, J101 TYPEC-305-ACP16H458, J501 GT-HD001B-CNNG1, J502 I2C, J503 SPI, J601 JST_SHBM04B-SRSS-TB, J701 Bus_M.2_Socket_M, J802 Conn_01x22_Female, M701 M.2 Solder Nut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

Commit message: SEEED
Parts:
- moved U401 4.01 mm to (101.5, 38.2)
- moved U402 4.01 mm to (101.5, 34.1)
Routing:
- net /CM5/ETH_PI.TRD2_N: track 46.2 -> 42.4 mm
- net /CM5/ETH_PI.TRD2_P: track 46.5 -> 42.6 mm
- net /CM5/ETH_PI.TRD3_P: track 46.3 -> 42.4 mm
- net /CM5/ETH_PI.TRD3_N: track 46.4 -> 42.6 mm
- net /CM5/ETH_PI.TRD1_N: track 46.1 -> 42.3 mm
- net /CM5/ETH_PI.TRD1_P: track 45.9 -> 42.1 mm
- net /CM5/ETH_PI.TRD0_N: track 45.2 -> 41.8 mm
- net /CM5/ETH_PI.TRD0_P: track 45.4 -> 42.0 mm
- net /CM5/PCIE_PI.nWAKE: track 39.4 -> 40.8 mm
- net /CM5/PCIE_PI.nRST: track 36.1 -> 37.4 mm
- net /CM5/PCIE_PI.nCLKREQ: track 40.4 -> 41.3 mm

Commit message: save
Other:
- board text removed: "PCB3D_BR_CM5_MINIMA_3"
- board text removed: "PCB3D_TL_CM5_MINIMA_3"
