File: CM5.kicad_sch (KiCad schematic)
At the start: 3 parts, among them M303 Compute-Module-4_H1.5mm

Commit message: DRC and prod files
Parts:
- added CN1: SM02B-SRSS-TB (LF)(SN), EasyEDA:CONN-SMD_2P-P1.00_SM02B-SRSS-TB-LF-SN, symbol EasyEDA:SM02B-SRSS-TB(LF)(SN)
Connections:
- net GND: now also CN1.2
- net VBAT renamed +BATT
- net +BATT: now also CN1.1
- no-connect marks 64 -> 67

Commit message: swapped I2C bus from 0 to 1
Connections:
- net GPIO2 renamed SDA1_IO2
- net GPIO3 renamed SCL1_IO3
Changed lines of the file:
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@@
 	(wire
 		(pts
-			(xy 71.12 147.32) (xy 86.36 147.32)
+			(xy 69.85 147.32) (xy 86.36 147.32)
 		)
 		(stroke
@@
 	(wire
 		(pts
-			(xy 71.12 149.86) (xy 86.36 149.86)
+			(xy 69.85 149.86) (xy 86.36 149.86)
 		)
 		(stroke
@@
 		)
 	)
-	(label "GPIO3"
-		(at 71.12 147.32 0)
-		(effects
-			(font
-				(size 1.27 1.27)
-			)
-			(justify left bottom)
-		)
-	)
 	(label "DPHY1_P.D3_P"
 		(at 251.46 200.66 0)
@@
 		)
 	)
-	(label "GPIO2"
-		(at 71.12 149.86 0)
-		(effects
-			(font
-				(size 1.27 1.27)
-			)
-			(justify left bottom)
-		)
-	)
 	(label "HDMI1_SDA"
 		(at 332.74 137.16 0)
@@
 		)
 	)
+	(hierarchical_label "SDA1_IO2"
+		(shape input)
+		(at 69.85 149.86 180)
+		(effects
+			(font
+				(size 1.27 1.27)
+			)
+			(justify right)
+		)
+	)
 	(hierarchical_label "PI_nLED_PWR"
 		(shape output)
@@
 		(effects
 			(font
+				(size 1.27 1.27)
+			)
+			(justify right)
+		)
+	)
+	(hierarchical_label "SCL1_IO3"
+		(shape input)
+		(at 69.85 147.32 180)
+		(effects
+			(font
