File: CM5_MINIMA_3.kicad_sch (KiCad schematic)
At the start: 18 parts, among them J101 TYPEC-305-ACP16H458, SW101 MK-11C04-G013

Commit message: arcs
Parts:
- added H102, H103, H104, H105: MountingHole_Pad, MountingHole:MountingHole_2.7mm_Pad, symbol Mechanical:MountingHole_Pad
Connections:
- net GND: now also H102.1, H103.1, H104.1, H105.1
Other:
- moved on the sheet: H101

Commit message: vias
Parts:
- R105, R106: now not fitted; now left out of the parts list
Changed lines of the file:
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@@
 		(unit 1)
 		(exclude_from_sim no)
-		(in_bom yes)
-		(on_board yes)
-		(dnp no)
+		(in_bom no)
+		(on_board yes)
+		(dnp yes)
 		(property "Reference" "R105"
 			(at 184.912 140.97 90)
@@
 		(unit 1)
 		(exclude_from_sim no)
-		(in_bom yes)
-		(on_board yes)
-		(dnp no)
+		(in_bom no)
+		(on_board yes)
+		(dnp yes)
 		(property "Reference" "R106"
 			(at 184.912 136.144 90)

Commit message: DRC and prod files
Parts:
- removed R105, R106: 0R, Resistor_SMD:R_0402_1005Metric, symbol Device:R
Other:
- sheet CM5 ports: added none; removed GPIO4, GPIO5
- sheet PCIe-M2 ports: added none; removed RX, TX

Commit message: swapped I2C bus from 0 to 1
Other:
- sheet CM5 ports: added SCL1_IO3, SDA1_IO2; removed none
- note added: "CHANGE LOG - swapped sensors' I2C from MIPI0 to I2C1 (IO56-58)"
- moved on the sheet: H101, H102, H103, H104, H105, SW101
