File: PCIe-M2.kicad_sch (KiCad schematic)
At the start: 22 parts, among them J701 Bus_M.2_Socket_M, M701 M.2 Solder Nut, M702 M.2 Solder Nut, M705 M.2 Screw, U702 AP3441SHE-7B, U703 ASEK-32.768KHZ-L-R-T

Commit message: vias
Connections:
- net M2_LX: now reaches L701.1, U702.6 (LX)
Changed lines of the file:
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@@
+		)
+	)
+	(label "M2_LX"
+		(at 83.82 167.64 0)
+		(effects
+			(font
+				(size 1.27 1.27)
+			)
+			(justify left bottom)
 		)
 	)

Commit message: DRC and prod files
Connections:
- net RX: no longer names the net of J701.22 (NC)
- net TX: no longer names the net of J701.20 (NC)
- no-connect marks 15 -> 17
Changed lines of the file:
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@@
+	)
+	(no_connect
+		(at 180.34 77.47)
 	)
 	(no_connect
@@
 	(no_connect
 		(at 180.34 100.33)
+	)
+	(no_connect
+		(at 180.34 74.93)
 	)
 	(no_connect
@@
 	(wire
 		(pts
-			(xy 180.34 77.47) (xy 185.42 77.47)
-		)
-		(stroke
-			(width 0)
-			(type default)
-		)
-	)
-	(wire
-		(pts
 			(xy 58.42 176.53) (xy 58.42 170.18)
 		)
@@
 			(width 0)
 			(type solid)
-		)
-	)
-	(wire
-		(pts
-			(xy 180.34 74.93) (xy 185.42 74.93)
-		)
-		(stroke
-			(width 0)
-			(type default)
 		)
 	)
@@
 		)
 	)
-	(hierarchical_label "TX"
-		(shape input)
-		(at 185.42 77.47 0)
-		(effects
-			(font
-				(size 1.27 1.27)
-			)
-			(justify left)
-		)
-	)
-	(hierarchical_label "RX"
-		(shape input)
-		(at 185.42 74.93 0)
-		(effects
-			(font
-				(size 1.27 1.27)
-			)
-			(justify left)
-		)
-	)
