File: USB.kicad_sch (KiCad schematic)
At the start: 9 parts, among them U701 AP22653W6

Commit message: vias
Parts:
- C702: footprint Capacitor_Tantalum_SMD:CP_EIA-7343-31_Kemet-D -> Capacitor_Tantalum_SMD:CP_EIA-3528-21_Kemet-B; Field4 Mouser -> (none); Field5 667-EEF-CX0J101R -> TAJB107K006RNJ; Field7 Panasonic -> (none); Part Description Capacitor, SP-Cap, 100u, 6.3V, 15mR ESR -> 100uF 6.3V 1.7Ω@100kHz ±10% CASE-B-3528-21(mm) Tantalum Cap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
Changed lines of the file:
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@@
 			)
 		)
-		(property "Footprint" "Capacitor_Tantalum_SMD:CP_EIA-7343-31_Kemet-D"
+		(property "Footprint" "Capacitor_Tantalum_SMD:CP_EIA-3528-21_Kemet-B"
 			(at 134.3152 46.99 0)
 			(effects
@@
 			)
 		)
-		(property "Field4" "Mouser"
+		(property "Field5" "TAJB107K006RNJ"
 			(at 133.35 43.18 0)
 			(effects
@@
 			)
 		)
-		(property "Field5" "667-EEF-CX0J101R"
+		(property "Part Description" " 100uF 6.3V 1.7Ω@100kHz ±10% CASE-B-3528-21(mm) Tantalum Capacitors ROHS"
 			(at 133.35 43.18 0)
 			(effects
-				(font
-					(size 1.27 1.27)
-				)
-				(hide yes)
-			)
-		)
-		(property "Part Description" "Capacitor, SP-Cap, 100u, 6.3V, 15mR ESR"
-			(at 133.35 43.18 0)
-			(effects
-				(font
-					(size 1.27 1.27)
-				)
-				(hide yes)
-			)
-		)
-		(property "Field7" "Panasonic"
-			(at 133.35 43.18 0)
-			(effects
